Commit message: Just added a note for the collision envelope of the robots.

File: urdf/robot_base.urdf (robot description, URDF)
Before this commit: robot puppeteer, 15 links, 14 joints
Links:
- link cover: geometry collision cylinder length=.14 radius=0.12; visual cylinder length=.1397 radius=.105
